File: HD3SS3220-breakout.kicad_sch (KiCad schematic)
At the start: 15 parts, among them J1 484050003, U1 HD3SS3220IRNHR, U2 MC-312D

Commit message: Reorganize library to follow KiCad naming conventions
Restructure the library into categorized directories following KiCad's
official library naming scheme. Symbols use .kicad_symdir directories,
footprints use .pretty directories, and 3D models use .3dshapes
directories, all grouped by component category (MCU_RaspberryPi,
MCU_WCH, Interface_USB, Sensor_Motion, Regulator_Linear, Memory_Flash,
Connector_USB, Connector, Device, Switch).

Footprint files and 3D models are renamed to match their chip/component
name for easier identification. Internal references (footprint names,
3D model paths, schematic lib_ids) are updated to match the new
structure.

Co-Authored-By: Claude Opus 4.6 <noreply@anthropic.com>
Parts:
- J1: footprint CONN_484050003_MOL -> Connector:Molex-0484050003; symbol Molex-0484050003:484050003 -> Connector:484050003
- U1: footprint RNH0030A -> Interface_USB:HD3SS3220IRNHR; symbol HD3SS3220IRNHR:HD3SS3220IRNHR -> Interface_USB:HD3SS3220IRNHR
- U2: footprint footprint:USB-C-SMD_MC-312D-C -> Connector_USB:MC-312D; symbol MC-312D:MC-312D -> Connector_USB:MC-312D
Connections:
- net GND: no longer J1.4 (GND), U1.12 (EN_MUX_N), U1.13 (GND), U1.28 (GND), U1.29 (EN_CC_N), U1.3 (CURRENT_MODE), U1.31 (PAD), U2.A1 (GND), U2.A12 (GND), U2.B1 (GND), U2.B12 (GND)
- net VBUS: no longer J1.1 (VBUS), U2.A4 (VBUS), U2.A9 (VBUS), U2.B4 (VBUS), U2.B9 (VBUS)
- net VCC 3.3V: no longer U1.8 (VCC33)
- net VCC 5V: no longer U1.30 (VDD5)
- net at C.1: no longer U2.B3 (SSTXN2)
- net at C.2: no longer U1.20 (TX2N)
- net at R.2: no longer U1.11 (DIR)
- net at C.1, R.2: no longer J1.7 (GND_DRAIN)
- net at C.2: no longer U1.16 (TX1N)
- net at C.2: no longer U1.17 (TX1P)
- net at C.2: no longer U1.21 (TX2P)
- net at R.1: no longer U1.5 (VBUS_DET)
- net at C.1: no longer U2.B2 (SSTXP2)
- net at C.1: no longer U2.A2 (SSTXP1)
- net at C.1: no longer U2.A3 (SSTXN1)
- new net: C.1, R.1
Changed lines of the file:
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@@
 	)
 	(symbol
-		(lib_id "HD3SS3220IRNHR:HD3SS3220IRNHR")
+		(lib_id "Interface_USB:HD3SS3220IRNHR")
 		(at 134.62 119.38 0)
 		(unit 1)
@@
 			)
 		)
-		(property "Footprint" "RNH0030A"
+		(property "Footprint" "Interface_USB:HD3SS3220IRNHR"
 			(at 134.62 119.38 0)
 			(effects
@@
 	)
 	(symbol
-		(lib_id "Molex-0484050003:484050003")
+		(lib_id "Connector:484050003")
 		(at 58.42 127 0)
 		(mirror y)
@@
 			)
 		)
-		(property "Footprint" "CONN_484050003_MOL"
+		(property "Footprint" "Connector:Molex-0484050003"
 			(at 50.038 124.46 0)
 			(effects
@@
 	)
 	(symbol
-		(lib_id "MC-312D:MC-312D")
+		(lib_id "Connector_USB:MC-312D")
 		(at 228.6 63.5 0)
 		(unit 1)
@@
 			)
 		)
-		(property "Footprint" "footprint:USB-C-SMD_MC-312D-C"
+		(property "Footprint" "Connector_USB:MC-312D"
 			(at 228.6 73.66 0)
 			(effects
