File: HD3SS3220-breakout.kicad_sch (KiCad schematic)
At the start: 32 parts, among them J1 USB_C_Receptacle, J2 U-A-39SS-Y-1, J3 A2541WV-2x4P, SW3 DSHP06TSGER_C3293146, U1 HD3SS3220RNHR, U2 TPD2EUSB30, U3 TPD4EUSB30, U4 HT7533-1_C14289

Commit message: Rerouted for new elements added (5 DRC errors left)
Parts:
- J1: footprint Interface_USB:USB-C-SMD_TYPE-C-USB-19 -> Interface_USB:USB-C-SMD_TYPEC-324G-BCP24; LCSC C2927039 -> C920230; Store Page https://www.lcsc.com/product-detail/C2927039.html -> https://www.lcsc.com/product-detail/C920230.html
Changed lines of the file:
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@@
 	)
 	(junction
+		(at 123.19 39.37)
+		(diameter 0)
+		(color 0 0 0 0)
+	)
+	(junction
 		(at 218.44 93.98)
 		(diameter 0)
@@
 	)
 	(junction
-		(at 123.19 39.37)
-		(diameter 0)
-		(color 0 0 0 0)
-	)
-	(junction
 		(at 21.59 146.05)
 		(diameter 0)
@@
 		)
 	)
+	(label "V_OUT"
+		(at 96.52 39.37 180)
+		(effects
+			(font
+				(size 1.27 1.27)
+			)
+			(justify right bottom)
+		)
+	)
 	(label "CC2"
 		(at 233.68 36.83 180)
@@
 		)
 	)
-	(label "V_OUT"
-		(at 96.52 39.37 180)
-		(effects
-			(font
-				(size 1.27 1.27)
-			)
-			(justify right bottom)
-		)
-	)
 	(label "PORT"
 		(at 72.39 151.13 0)
@@
 			)
 		)
-		(property "Datasheet" ""
+		(property "Datasheet" "https://ds.yuden.co.jp/TYCOMPAS/ut/detail?pn=MSASE32MAB5107MPNA01&u=M"
 			(at 105.41 27.94 0)
 			(hide yes)
@@
 			)
 		)
-		(property "Footprint" "Interface_USB:USB-C-SMD_TYPE-C-USB-19"
+		(property "Footprint" "Interface_USB:USB-C-SMD_TYPEC-324G-BCP24"
 			(at 260.35 55.88 0)
 			(hide yes)
@@
 			)
 		)
-		(property "Store Page" "https://www.lcsc.com/product-detail/C2927039.html"
+		(property "Store Page" "https://www.lcsc.com/product-detail/C920230.html"
 			(at 264.16 55.88 0)
 			(hide yes)
@@
 			)
 		)
-		(property "LCSC" "C2927039"
+		(property "LCSC" "C920230"
 			(at 264.16 55.88 0)
 			(hide yes)
@@
 			)
 		)
-		(property "Datasheet" ""
+		(property "Datasheet" "https://yageogroup.com/products/Capacitors/part/CC0402KRX5R7BB104"
 			(at 105.41 43.18 0)
 			(hide yes)

Commit message: Generated Gerber files and proper BOM
Parts:
- TP1, TP2, TP3, TP4, TP5, TP6, TP7: now not fitted
- renumbered C7 to C1, C8 to C2, C11 to C3, C9 to C4, C12 to C5, C10 to C6, SW3 to SW1
Changed lines of the file:
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@@
 		(title "USB-3.0 Bridging Board Root")
 		(date "2026-04-16")
-		(rev "R1")
+		(rev "R3")
 		(company "UWaterloo Reality Labs")
 		(comment 4 "Authors: Brandon, Marcus, Dinh")
@@
 	(text "Bypass"
 		(exclude_from_sim no)
-		(at 94.996 30.988 0)
+		(at 94.996 30.734 0)
 		(effects
 			(font
@@
 		(on_board yes)
 		(in_pos_files yes)
-		(dnp no)
+		(dnp yes)
 		(property "Reference" "TP1"
 			(at 126.492 34.29 90)
@@
 		(on_board yes)
 		(in_pos_files yes)
-		(dnp no)
+		(dnp yes)
 		(property "Reference" "TP7"
 			(at 212.09 27.1779 0)
@@
 		(in_pos_files yes)
 		(dnp no)
-		(property "Reference" "C8"
+		(property "Reference" "C2"
 			(at 62.738 36.068 0)
 			(show_name no)
@@
 			(project "HD3SS3220-breakout"
 				(path "/6d9920bc-ffe5-49c6-a5b8-424c0488cfb7"
-					(reference "C8")
+					(reference "C2")
 					(unit 1)
 				)
@@
 		(in_pos_files yes)
 		(dnp no)
-		(property "Reference" "C9"
+		(property "Reference" "C4"
 			(at 97.282 41.148 0)
 			(show_name no)
@@
 			(project "HD3SS3220-breakout"
 				(path "/6d9920bc-ffe5-49c6-a5b8-424c0488cfb7"
-					(reference "C9")
+					(reference "C4")
 					(unit 1)
 				)
@@
 		(in_pos_files yes)
 		(dnp no)
-		(property "Reference" "SW3"
+		(property "Reference" "SW1"
 			(at 41.148 142.24 0)
 			(show_name no)
@@
 			(project "HD3SS3220-breakout"
 				(path "/6d9920bc-ffe5-49c6-a5b8-424c0488cfb7"
-					(reference "SW3")
+					(reference "SW1")
 					(unit 1)
 				)
@@
 		(on_board yes)
 		(in_pos_files yes)
-		(dnp no)
+		(dnp yes)
 		(property "Reference" "TP2"
 			(at 130.81 58.928 90)
@@
 		(on_board yes)
 		(in_pos_files yes)
-		(dnp no)
+		(dnp yes)
 		(property "Reference" "TP3"
 			(at 118.11 36.068 90)
@@
 		(on_board yes)
 		(in_pos_files yes)
-		(dnp no)
+		(dnp yes)
 		(property "Reference" "TP4"
 			(at 223.0121 92.71 0)
@@
 		(on_board yes)
 		(in_pos_files yes)
-		(dnp no)
+		(dnp yes)
 		(property "Reference" "TP6"
 			(at 209.55 27.1779 0)
@@
 		(on_board yes)
 		(in_pos_files yes)
-		(dnp no)
+		(dnp yes)
 		(property "Reference" "TP5"
 			(at 223.0121 96.52 0)
@@
 		(in_pos_files yes)
 		(dnp no)
-		(property "Reference" "C12"
-			(at 109.22 26.67 0)
+		(property "Reference" "C5"
+			(at 108.458 26.67 0)
 			(show_name no)
 			(do_not_autoplace no)
@@
 			(project "HD3SS3220-breakout"
 				(path "/6d9920bc-ffe5-49c6-a5b8-424c0488cfb7"
-					(reference "C12")
+					(reference "C5")
 					(unit 1)
 				)
@@
 		(in_pos_files yes)
 		(dnp no)
-		(property "Reference" "C7"
+		(property "Reference" "C1"
 			(at 26.924 36.068 0)
 			(show_name no)
@@
 			(project "HD3SS3220-breakout"
 				(path "/6d9920bc-ffe5-49c6-a5b8-424c0488cfb7"
-					(reference "C7")
+					(reference "C1")
 					(unit 1)
 				)
@@
 		(in_pos_files yes)
 		(dnp no)
-		(property "Reference" "C11"
-			(at 96.774 26.924 0)
+		(property "Reference" "C3"
+			(at 96.774 26.67 0)
 			(show_name no)
 			(do_not_autoplace no)
@@
 		)
 		(property "Value" "100nF"
-			(at 95.504 28.702 0)
+			(at 95.504 28.448 0)
 			(show_name no)
 			(do_not_autoplace no)
@@
 			(project "HD3SS3220-breakout"
 				(path "/6d9920bc-ffe5-49c6-a5b8-424c0488cfb7"
-					(reference "C11")
+					(reference "C3")
 					(unit 1)
 				)
@@
 		(in_pos_files yes)
 		(dnp no)
-		(property "Reference" "C10"
-			(at 109.22 41.148 0)
+		(property "Reference" "C6"
+			(at 108.712 41.148 0)
 			(show_name no)
 			(do_not_autoplace no)
@@
 			(project "HD3SS3220-breakout"
 				(path "/6d9920bc-ffe5-49c6-a5b8-424c0488cfb7"
-					(reference "C10")
+					(reference "C6")
 					(unit 1)
 				)

Commit message: Corrected ESD Diodes logic
Parts:
- removed U2: TPD2EUSB30, Package_TO_SOT_SMD:Texas_DRT-3, symbol Power_Protection:TPD2EUSB30
- added U2, U3: TPD4EUSB30, Package_SON:USON-10_2.5x1.0mm_P0.5mm, symbol Power_Protection:TPD4EUSB30
- renumbered U3 to U4, U4 to U5
Connections:
- net GND: now also U2.3 (GND), U2.8 (GND), U3.3 (GND), U3.8 (GND)
- net RX1+: now also U2.4 (D2+), U2.7 (NC)
- net RX1-: now also U2.5 (D2-), U2.6 (NC)
- net RX2+: now also U3.4 (D2+), U3.7 (NC)
- net RX2-: now also U3.5 (D2-), U3.6 (NC)
- net TX1+: now also U2.2 (D1-), U2.9 (NC)
- net TX1-: now also U2.1 (D1+), U2.10 (NC)
- net TX2+: now also U3.1 (D1+), U3.10 (NC)
- net TX2-: now also U3.2 (D1-), U3.9 (NC)
Other:
- moved on the sheet: C3, C4, C5, C6, J1, J2, R1, R2, R3, R4, R5, R6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
