File: HD3SS3220-breakout.kicad_sch (KiCad schematic)
At the start: 33 parts, among them J1 USB_C_Receptacle, J2 U-A-39SS-Y-1, J3 A2541WV-2x4P, SW1 DSHP06TSGER_C3293146, U1 HD3SS3220RNHR, U2 TPD4EUSB30, U3 TPD4EUSB30, U4 TPD4EUSB30, U5 HT7533-1_C14289

Commit message: Via to Ground Pour Clearance Fixed, D+/D- Lines Split Shortened, Ground Stitching Added, Other Symbols and Footprint Changed
Parts:
- TP1, TP2, TP3, TP6, TP7: footprint TestPoint:TestPoint_Pad_D1.5mm -> TestPoint:TestPoint_Keystone_5000-5004_Miniature
Connections:
- net V_OUT: now reaches C2.1, C4.2, C6.2, R2.1, R7.1, R9.1, TP3.1, U1.8 (VCC33), U5.3 (Vout)
Changed lines of the file:
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@@
 	(wire
 		(pts
-			(xy 60.96 30.48) (xy 66.04 30.48)
-		)
-		(stroke
-			(width 0)
-			(type default)
-		)
-	)
-	(wire
-		(pts
 			(xy 91.44 138.43) (xy 93.98 138.43)
 		)
@@
 	(wire
 		(pts
+			(xy 60.96 30.48) (xy 66.04 30.48)
+		)
+		(stroke
+			(width 0)
+			(type default)
+		)
+	)
+	(wire
+		(pts
 			(xy 242.57 132.08) (xy 245.11 132.08)
 		)
@@
 		)
 	)
+	(wire
+		(pts
+			(xy 66.04 27.94) (xy 66.04 30.48)
+		)
+		(stroke
+			(width 0)
+			(type default)
+		)
+	)
 	(polyline
 		(pts
@@
 	(wire
 		(pts
+			(xy 90.17 38.1) (xy 90.17 39.37)
+		)
+		(stroke
+			(width 0)
+			(type default)
+		)
+	)
+	(wire
+		(pts
 			(xy 21.59 156.21) (xy 21.59 154.94)
 		)
@@
 	(wire
 		(pts
+			(xy 90.17 39.37) (xy 116.84 39.37)
+		)
+		(stroke
+			(width 0)
+			(type default)
+		)
+	)
+	(wire
+		(pts
 			(xy 57.15 72.39) (xy 60.96 72.39)
 		)
@@
 	(wire
 		(pts
-			(xy 90.17 39.37) (xy 116.84 39.37)
-		)
-		(stroke
-			(width 0)
-			(type default)
-		)
-	)
-	(wire
-		(pts
 			(xy 242.57 45.72) (xy 242.57 43.18)
 		)
@@
 		)
 	)
-	(label "V_OUT"
-		(at 66.04 30.48 0)
-		(effects
-			(font
-				(size 1.27 1.27)
-			)
-			(justify left bottom)
-		)
-	)
 	(label "RX1+"
 		(at 228.6 121.92 0)
@@
 		)
 	)
-	(label "V_OUT"
-		(at 90.17 39.37 180)
-		(effects
-			(font
-				(size 1.27 1.27)
-			)
-			(justify right bottom)
-		)
-	)
 	(label "TX1-"
 		(at 198.12 127 180)
@@
 			)
 		)
-		(property "Footprint" "TestPoint:TestPoint_Pad_D1.5mm"
+		(property "Footprint" "TestPoint:TestPoint_Keystone_5000-5004_Miniature"
 			(at 116.84 34.29 0)
 			(hide yes)
@@
 	)
 	(symbol
+		(lib_id "power:VBUS")
+		(at 90.17 38.1 0)
+		(unit 1)
+		(body_style 1)
+		(exclude_from_sim no)
+		(in_bom yes)
+		(on_board yes)
+		(in_pos_files yes)
+		(dnp no)
+		(property "Reference" "#PWR027"
+			(at 90.17 41.91 0)
+			(hide yes)
+			(show_name no)
+			(do_not_autoplace no)
+			(effects
+				(font
+					(size 1.27 1.27)
+				)
+			)
+		)
+		(property "Value" "V_OUT"
+			(at 86.106 37.084 0)
+			(show_name no)
+			(do_not_autoplace no)
+			(effects
+				(font
+					(size 1.27 1.27)
+				)
+			)
+		)
+		(property "Footprint" ""
+			(at 90.17 38.1 0)
+			(hide yes)
+			(show_name no)
+			(do_not_autoplace no)
+			(effects
+				(font
+					(size 1.27 1.27)
+				)
+			)
+		)
+		(property "Datasheet" ""
+			(at 90.17 38.1 0)
+			(hide yes)
+			(show_name no)
+			(do_not_autoplace no)
+			(effects
+				(font
+					(size 1.27 1.27)
+				)
+			)
+		)
+		(property "Description" "Power symbol creates a global label with name \"VBUS\""
+			(at 90.17 38.1 0)
+			(hide yes)
+			(show_name no)
+			(do_not_autoplace no)
+			(effects
+				(font
+					(size 1.27 1.27)
+				)
+			)
+		)
+		(pin "1"
+		)
+		(instances
+			(project "HD3SS3220-breakout"
+				(path "/6d9920bc-ffe5-49c6-a5b8-424c0488cfb7"
+					(reference "#PWR027")
+					(unit 1)
+				)
+			)
+		)
+	)
+	(symbol
 		(lib_id "Connector_USB-custom:U-A-39SS-Y-1")
 		(at 157.48 134.62 0)
@@
 			)
 		)
-		(property "Footprint" "TestPoint:TestPoint_Pad_D1.5mm"
+		(property "Footprint" "TestPoint:TestPoint_Keystone_5000-5004_Miniature"
 			(at 208.28 31.75 0)
 			(hide yes)
@@
 			)
 		)
-		(property "Footprint" "TestPoint:TestPoint_Pad_D1.5mm"
+		(property "Footprint" "TestPoint:TestPoint_Keystone_5000-5004_Miniature"
 			(at 124.46 62.23 0)
 			(hide yes)
@@
 			)
 		)
-		(property "Footprint" "TestPoint:TestPoint_Pad_D1.5mm"
+		(property "Footprint" "TestPoint:TestPoint_Keystone_5000-5004_Miniature"
 			(at 111.76 39.37 0)
 			(hide yes)
@@
 	)
 	(symbol
+		(lib_id "power:VBUS")
+		(at 66.04 27.94 0)
+		(unit 1)
+		(body_style 1)
+		(exclude_from_sim no)
+		(in_bom yes)
+		(on_board yes)
+		(in_pos_files yes)
+		(dnp no)
+		(property "Reference" "#PWR040"
+			(at 66.04 31.75 0)
+			(hide yes)
+			(show_name no)
+			(do_not_autoplace no)
+			(effects
+				(font
+					(size 1.27 1.27)
+				)
+			)
+		)
+		(property "Value" "V_OUT"
+			(at 70.104 26.67 0)
+			(show_name no)
+			(do_not_autoplace no)
+			(effects
+				(font
+					(size 1.27 1.27)
+				)
+			)
+		)
+		(property "Footprint" ""
+			(at 66.04 27.94 0)
+			(hide yes)
+			(show_name no)
+			(do_not_autoplace no)
+			(effects
+				(font
+					(size 1.27 1.27)
+				)
+			)
+		)
+		(property "Datasheet" ""
+			(at 66.04 27.94 0)
+			(hide yes)
+			(show_name no)
+			(do_not_autoplace no)
+			(effects
+				(font
+					(size 1.27 1.27)
+				)
+			)
+		)
+		(property "Description" "Power symbol creates a global label with name \"VBUS\""
+			(at 66.04 27.94 0)
+			(hide yes)
+			(show_name no)
+			(do_not_autoplace no)
+			(effects
+				(font
+					(size 1.27 1.27)
+				)
+			)
+		)
+		(pin "1"
+		)
+		(instances
+			(project "HD3SS3220-breakout"
+				(path "/6d9920bc-ffe5-49c6-a5b8-424c0488cfb7"
+					(reference "#PWR040")
+					(unit 1)
+				)
+			)
+		)
+	)
+	(symbol
 		(lib_id "Device:LED")
 		(at 44.45 119.38 90)
@@
 			)
 		)
-		(property "Footprint" "TestPoint:TestPoint_Pad_D1.5mm"
+		(property "Footprint" "TestPoint:TestPoint_Keystone_5000-5004_Miniature"
 			(at 205.74 31.75 0)
 			(hide yes)

Commit message: Footprint and symbol fix
Parts:
- J1: symbol Connector:USB_C_Receptacle -> UWRealityLabs:TYPEC-324G-BCP24
Connections:
- net GND: now also J1.1 (EP), J1.2 (EP), J1.3 (EP), J1.4 (EP); no longer J1.S1 (SHIELD)
Other:
- note removed: "power flags"
- note removed: "rule area for marking impedence match pairs"
- note removed: "watch videos on high speed routing for ki cad specifically"
- moved on the sheet: C1, C2, C3, C4, C5, C6, DIR_LED2, J2, J3, R1, R2, R3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

Commit message: Regenerate all Production/ outputs from the repaired board
The previous set was self-contradictory and unfabricatable: gerbers exported
from the pre-fix board still contained the VBUS=GND dead short, netlist.ipc
was from Jul 7 (pre-corruption refs), bom.xlsx was from Jun 15 (stale refs,
LDO/ESD collision), and no pick-and-place existed at all.

All outputs now come from one board revision, exported with the board's own
plot parameters (same layer set and names):
- gerbers + Excellon PTH/NPTH + HD3SS3220-gerbers.zip (same 19-file recipe)
- netlist.ipc: fresh IPC-D-356
- bom.csv (replaces stale bom.xlsx): 25 grouped rows from schematic fields;
  R5 LCSC consolidated to C413111 to match R6/R7 (same 10K 0402, one SKU)
- HD3SS3220-breakout-cpl.csv: pick-and-place, previously missing

F.Cu gerber VBUS-attributed objects: 3 (shorted export) -> 18.
Parts:
- R5: LCSC C4326584 -> C413111
Changed lines of the file:
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@@
 			)
 		)
-		(property "LCSC" "C4326584"
+		(property "LCSC" "C413111"
 			(at 62.23 144.78 90)
 			(hide yes)
