File: HD3SS3220-breakout.kicad_pcb (KiCad board)
At the start: 4 copper layers, 29 x 53.3 mm, 34 parts, among them J1 USB_C_Receptacle, J2 U-A-39SS-Y-1, J3 A2541WV-2x4P, SW3 DSHP06TSGER_C3293146, U1 HD3SS3220RNHR, U2 TPD2EUSB30, U3 TPD4EUSB30, U4 HT7533-1_C14289

Commit message: Generated Gerber files and proper BOM
Parts:
- renumbered C7 to C1, C8 to C2, C11 to C3, C09 to C4, C12 to C5, C10 to C6, SW3 to SW1, V_OUT to TP3
Connections:
- J1 pad : GND -> (no net)
- J1 pad 1: GND -> (no net)
- J1 pad 2: GND -> (no net)
- J1 pad 3: GND -> (no net)
- J1 pad 4: GND -> (no net)
Other:
- board text added: "UWaterloo Reality Labs"
Changed lines of the file:
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@@
 		(tags "USON-10 2.5x1.0mm Pitch 0.5mm")
 		(property "Reference" "U3"
-			(at 0.01829 -2.5 90)
+			(at 0.015 2 90)
 			(layer "F.SilkS")
 			(effects
 				(font
-					(size 1 1)
-					(thickness 0.15)
+					(size 0.75 0.75)
 				)
 			)
@@
 			(layers "F.Cu" "F.Mask" "F.Paste")
 			(roundrect_rratio 0.25)
-			(net "Net-(SW3-A3)")
+			(net "Net-(SW1-A3)")
 			(pintype "passive")
 		)
@@
 		(descr "Capacitor SMD 1210 (3225 Metric), square (rectangular) end terminal, IPC-7351 nominal, (Body size source: IPC-SM-782 page 76, https://www.pcb-3d.com/wordpress/wp-content/uploads/ipc-sm-782a_amendment_1_and_2.pdf)")
 		(tags "capacitor")
-		(property "Reference" "C12"
+		(property "Reference" "C5"
 			(at -1.325 -2.2 270)
 			(layer "F.SilkS")
@@
 		(descr "Capacitor SMD 0402 (1005 Metric), square (rectangular) end terminal, IPC-7351 nominal, (Body size source: IPC-SM-782 page 76, https://www.pcb-3d.com/wordpress/wp-content/uploads/ipc-sm-782a_amendment_1_and_2.pdf)")
 		(tags "capacitor")
-		(property "Reference" "C10"
+		(property "Reference" "C6"
 			(at 2.08 -0.8 0)
 			(layer "F.SilkS")
@@
 		(tags "DRT-3 1x0.8mm Pitch 0.7mm")
 		(property "Reference" "U2"
-			(at 0 -1.5 90)
+			(at 1.6 0 90)
 			(layer "F.SilkS")
 			(effects
 				(font
-					(size 1 1)
-					(thickness 0.15)
+					(size 0.75 0.75)
 				)
 			)
@@
 			(layers "F.Cu" "F.Mask" "F.Paste")
 			(roundrect_rratio 0.25)
-			(net "Net-(SW3-B2)")
+			(net "Net-(SW1-B2)")
 			(pintype "passive")
 		)
@@
 		(descr "SMD pad as test Point, diameter 1.5mm")
 		(tags "test point SMD pad")
-		(property "Reference" "V_OUT"
+		(property "Reference" "TP3"
 			(at 2 -0.1 90)
 			(layer "F.SilkS")
@@
 		(layer "F.Cu")
 		(at 117.2 53.6 90)
-		(property "Reference" "SW3"
+		(property "Reference" "SW1"
 			(at 5.47 -1.49 180)
 			(layer "F.SilkS")
@@
 			(size 1.27 0.762)
 			(layers "F.Cu" "F.Mask" "F.Paste")
-			(net "Net-(SW3-A3)")
+			(net "Net-(SW1-A3)")
 			(pinfunction "A3_3")
 			(pintype "passive")
@@
 			(size 1.27 0.762)
 			(layers "F.Cu" "F.Mask" "F.Paste")
-			(net "Net-(SW3-B2)")
+			(net "Net-(SW1-B2)")
 			(pinfunction "B2_11")
 			(pintype "passive")
@@
 			(size 1.27 0.762)
 			(layers "F.Cu" "F.Mask" "F.Paste")
-			(net "Net-(SW3-B1)")
+			(net "Net-(SW1-B1)")
 			(pinfunction "B1_12")
 			(pintype "passive")
@@
 		(descr "Capacitor SMD 0402 (1005 Metric), square (rectangular) end terminal, IPC-7351 nominal, (Body size source: IPC-SM-782 page 76, https://www.pcb-3d.com/wordpress/wp-content/uploads/ipc-sm-782a_amendment_1_and_2.pdf)")
 		(tags "capacitor")
-		(property "Reference" "C8"
-			(at -1.78 0 0)
+		(property "Reference" "C2"
+			(at -1.58 -0.1 90)
 			(layer "F.SilkS")
 			(effects
@@
 		(descr "Capacitor SMD 0402 (1005 Metric), square (rectangular) end terminal, IPC-7351 nominal, (Body size source: IPC-SM-782 page 76, https://www.pcb-3d.com/wordpress/wp-content/uploads/ipc-sm-782a_amendment_1_and_2.pdf)")
 		(tags "capacitor")
-		(property "Reference" "C09"
+		(property "Reference" "C4"
 			(at 2.08 -0.8 0)
 			(layer "F.SilkS")
@@
 		(descr "Capacitor SMD 0402 (1005 Metric), square (rectangular) end terminal, IPC-7351 nominal, (Body size source: IPC-SM-782 page 76, https://www.pcb-3d.com/wordpress/wp-content/uploads/ipc-sm-782a_amendment_1_and_2.pdf)")
 		(tags "capacitor")
-		(property "Reference" "C11"
+		(property "Reference" "C3"
 			(at -2 0 270)
 			(layer "F.SilkS")
@@
 		(at 98.36 54.2 180)
 		(property "Reference" "U4"
-			(at -1.16 3.2 0)
+			(at -2.64 1.8 90)
 			(layer "F.SilkS")
 			(effects
 				(font
-					(size 1 1)
-					(thickness 0.15)
+					(size 0.75 0.75)
 				)
 			)
@@
 		(sheetname "/")
 		(sheetfile "HD3SS3220-breakout.kicad_sch")
+		(units
+			(unit
+				(name "A")
+				(pins "S1" "B1" "B12" "A1" "A12" "B9" "A9" "B4" "A4" "A5" "B5" "A7" "B7"
+					"A6" "B6" "B10" "B11" "A3" "A2" "A10" "A11" "B3" "B2" "A8" "B8"
+				)
+			)
+		)
 		(attr smd)
 		(duplicate_pad_numbers_are_jumpers no)
@@
 			(layers "*.Cu" "*.Mask")
 			(remove_unused_layers no)
-			(net "GND")
 		)
 		(pad "" thru_hole circle
@@
 			(layers "*.Cu" "*.Mask")
 			(remove_unused_layers no)
-			(net "GND")
 		)
 		(pad "1" thru_hole oval
@@
 			(layers "*.Cu" "*.Mask")
 			(remove_unused_layers no)
-			(net "GND")
 		)
 		(pad "1" thru_hole oval
@@
 			(layers "*.Cu" "*.Mask")
 			(remove_unused_layers no)
-			(net "GND")
 		)
 		(pad "2" thru_hole oval
@@
 			(layers "*.Cu" "*.Mask")
 			(remove_unused_layers no)
-			(net "GND")
 		)
 		(pad "2" thru_hole oval
@@
 			(layers "*.Cu" "*.Mask")
 			(remove_unused_layers no)
-			(net "GND")
 		)
 		(pad "3" thru_hole oval
@@
 			(layers "*.Cu" "*.Mask")
 			(remove_unused_layers no)
-			(net "GND")
 		)
 		(pad "4" thru_hole oval
@@
 			(layers "*.Cu" "*.Mask")
 			(remove_unused_layers no)
-			(net "GND")
 		)
 		(pad "A1" smd rect
@@
 		(descr "Capacitor SMD 0402 (1005 Metric), square (rectangular) end terminal, IPC-7351 nominal, (Body size source: IPC-SM-782 page 76, https://www.pcb-3d.com/wordpress/wp-content/uploads/ipc-sm-782a_amendment_1_and_2.pdf)")
 		(tags "capacitor")
-		(property "Reference" "C7"
+		(property "Reference" "C1"
 			(at 1.72 -0.08 90)
 			(layer "F.SilkS")
@@
 		(sheetname "/")
 		(sheetfile "HD3SS3220-breakout.kicad_sch")
+		(units
+			(unit
+				(name "A")
+				(pins "30" "8" "5" "29" "11" "23" "27" "22" "4" "24" "3" "25" "26" "6"
+					"7" "9" "10" "2" "1" "12" "17" "16" "15" "14" "21" "20" "19" "18" "28"
+					"13" "31"
+				)
+			)
+		)
 		(attr smd)
 		(duplicate_pad_numbers_are_jumpers no)
@@
 			(remove_unused_layers no)
 			(net "GND")
+			(pinfunction "EP_31")
+			(pintype "input")
 		)
 		(pad "31" thru_hole circle
@@
 			(remove_unused_layers no)
 			(net "GND")
+			(pinfunction "EP_31")
+			(pintype "input")
 		)
 		(pad "31" thru_hole circle
@@
 			(remove_unused_layers no)
 			(net "GND")
+			(pinfunction "EP_31")
+			(pintype "input")
 		)
 		(pad "31" smd rect
@@
 			(remove_unused_layers no)
 			(net "GND")
+			(pinfunction "EP_31")
+			(pintype "input")
 		)
 		(pad "31" thru_hole circle
@@
 			(remove_unused_layers no)
 			(net "GND")
+			(pinfunction "EP_31")
+			(pintype "input")
 		)
 		(pad "31" thru_hole circle
@@
 			(remove_unused_layers no)
 			(net "GND")
+			(pinfunction "EP_31")
+			(pintype "input")
 		)
 		(embedded_fonts no)
@@
 			(layers "F.Cu" "F.Mask" "F.Paste")
 			(roundrect_rratio 0.243902)
-			(net "Net-(SW3-B1)")
+			(net "Net-(SW1-B1)")
 			(pintype "passive")
 		)
@@
 		)
 	)
+	(gr_text "UWaterloo\nReality\nLabs"
+		(at 98.6 82.5 90)
+		(layer "F.SilkS")
+		(effects
+			(font
+				(size 0.75 0.75)
+				(bold yes)
+			)
+			(justify left bottom)
+		)
+	)
 	(gr_text "Brandon T,\nDinh L,\nMarcus L,"
-		(at 98.8 83.2 90)
+		(at 100.8 75 90)
 		(layer "F.SilkS")
 		(effects
@@
 	)
 	(via
-		(at 97 78.75)
+		(at 97 77.2)
 		(size 0.6)
 		(drill 0.3)
@@
 		(width 0.2)
 		(layer "F.Cu")
-		(net "Net-(SW3-A3)")
+		(net "Net-(SW1-A3)")
 	)
 	(segment
@@
 		(width 0.2)
 		(layer "F.Cu")
-		(net "Net-(SW3-A3)")
+		(net "Net-(SW1-A3)")
 	)
 	(segment
@@
 		(width 0.2)
 		(layer "F.Cu")
-		(net "Net-(SW3-A3)")
+		(net "Net-(SW1-A3)")
 	)
 	(segment
@@
 		(width 0.2)
 		(layer "F.Cu")
-		(net "Net-(SW3-B2)")
+		(net "Net-(SW1-B2)")
 	)
 	(segment
@@
 		(width 0.2)
 		(layer "F.Cu")
-		(net "Net-(SW3-B2)")
+		(net "Net-(SW1-B2)")
 	)
 	(segment
@@
 		(width 0.2)
 		(layer "F.Cu")
-		(net "Net-(SW3-B1)")
+		(net "Net-(SW1-B1)")
 	)
 	(segment
@@
 		(width 0.2)
 		(layer "F.Cu")
-		(net "Net-(SW3-B1)")
+		(net "Net-(SW1-B1)")
 	)
 	(segment
